Commit message: update 22/10 - hand tracking bugs&fixes

File: robot_hand_ws/src/robot_hand_description/urdf/hand.urdf.xacro (robot description, xacro)
@@ -13,5 +13,23 @@
     <visual>
       <geometry>
-        <box size="0.09 0.02 0.11"/>
+        <mesh filename="package://robot_hand_description/meshes/palm.stl"/>
+      </geometry>
+      <material name="blue"/>
+    </visual>
+  </link>
+  <!-- CMC opposition carries the blue pad and every downstream thumb joint. -->
+  <joint name="thumb_opposition" type="revolute">
+    <parent link="palm"/>
+    <child link="thenar"/>
+    <origin xyz="0.018 0 -0.035"/>
+    <axis xyz="0 0 -1"/>
+    <limit lower="0" upper="1.2" effort="1" velocity="1"/>
+  </joint>
+  <link name="thenar">
+    <!-- Offset preserves the pad's existing resting placement. -->
+    <visual name="thumb_pad">
+      <origin xyz="-0.018 0 0.035"/>
+      <geometry>
+        <mesh filename="package://robot_hand_description/meshes/thumb_pad.stl"/>
       </geometry>
       <material name="blue"/>
@@ -21,4 +39,13 @@
   <xacro:macro name="finger"
                params="name x z l1 l2 l3 angle:=0">
+    <!-- Abduction/adduction precedes flexion at the same MCP pivot. -->
+    <link name="${name}_knuckle"/>
+    <joint name="${name}_spread" type="revolute">
+      <parent link="palm"/>
+      <child link="${name}_knuckle"/>
+      <origin xyz="${x} 0 ${z}" rpy="0 ${angle} 0"/>
+      <axis xyz="0 1 0"/>
+      <limit lower="-0.45" upper="0.45" effort="1" velocity="1"/>
+    </joint>
     <!-- Proximal segment -->
     <link name="${name}_proximal">
@@ -32,7 +59,6 @@
     </link>
     <joint name="${name}_mcp" type="revolute">
-      <parent link="palm"/>
+      <parent link="${name}_knuckle"/>
       <child link="${name}_proximal"/>
-      <origin xyz="${x} 0 ${z}" rpy="0 ${angle} 0"/>
       <axis xyz="1 0 0"/>
       <limit lower="0" upper="1.57"
@@ -89,10 +115,19 @@
                 x="-0.032" z="0.055"
                 l1="0.035" l2="0.020" l3="0.015"/>
+  <!-- Sideways thumb rotation is independent from the two existing bends. -->
+  <link name="thumb_knuckle"/>
+  <joint name="thumb_spread" type="revolute">
+    <parent link="thenar"/>
+    <child link="thumb_knuckle"/>
+    <origin xyz="0.034 -0.006 0.042" rpy="0 0.9 0"/>
+    <axis xyz="0 1 0"/>
+    <limit lower="-0.8" upper="0.8" effort="1" velocity="1"/>
+  </joint>
   <!-- Simplified two-segment thumb -->
   <link name="thumb_proximal">
     <visual>
-      <origin xyz="0 0 0.023"/>
+      <origin xyz="0 0 0.0175"/>
       <geometry>
-        <box size="0.020 0.020 0.046"/>
+        <box size="0.022 0.022 0.035"/>
       </geometry>
       <material name="gray"/>
@@ -100,8 +135,6 @@
   </link>
   <joint name="thumb_base" type="revolute">
-    <parent link="palm"/>
+    <parent link="thumb_knuckle"/>
     <child link="thumb_proximal"/>
-    <origin xyz="0.045 0 0.005"
-            rpy="0 0.9 0"/>
     <axis xyz="1 0 0"/>
     <limit lower="0" upper="1.57"
@@ -110,7 +143,7 @@
   <link name="thumb_distal">
     <visual>
-      <origin xyz="0 0 0.025"/>
+      <origin xyz="0 0 0.013"/>
       <geometry>
-        <box size="0.018 0.018 0.050"/>
+        <box size="0.020 0.020 0.026"/>
       </geometry>
       <material name="gray"/>
@@ -120,5 +153,5 @@
     <parent link="thumb_proximal"/>
     <child link="thumb_distal"/>
-    <origin xyz="0 0 0.046"/>
+    <origin xyz="0 0 0.035"/>
     <axis xyz="1 0 0"/>
     <limit lower="0" upper="1.4"
